File: ENYA-SIMR-GTWL-PCTB.kicad_pcb (KiCad board)
At the start: 2 copper layers, 57.6 x 21.4 mm, 15 parts, among them J1 PICO_BLADE_1x5_MALE_RA_SMD, J2 PICO_BLADE_1x5_MALE_RA_SMD, SW1 SKSTAJE010, SW2 SKSTAJE010, SW3 SKSTAJE010, SW4 SKSTAJE010, SW5 SKSTAJE010, SW6 SKSTAJE010

Commit message: correction button matrix diode polarity
Parts:
- turned D1 to 0 degrees
- turned D2 to 180 degrees
- turned D3 to 180 degrees
Connections:
- D1 pad 1: /BTN_ROW0 -> Net-(D1-K)
- D1 pad 2: Net-(D1-A) -> /BTN_ROW0
- D2 pad 1: /BTN_ROW1 -> Net-(D2-K)
- D2 pad 2: Net-(D2-A) -> /BTN_ROW1
- D3 pad 1: /BTN_ROW2 -> Net-(D3-K)
- D3 pad 2: Net-(D3-A) -> /BTN_ROW2
- SW1 pad 2: Net-(D1-A) -> Net-(D1-K)
- SW2 pad 2: Net-(D1-A) -> Net-(D1-K)
- SW3 pad 2: Net-(D2-A) -> Net-(D2-K)
- SW4 pad 2: Net-(D2-A) -> Net-(D2-K)
- SW5 pad 2: Net-(D3-A) -> Net-(D3-K)
- SW6 pad 2: Net-(D3-A) -> Net-(D3-K)
Routing:
- net Net-(D3-K): track 0.00 -> 10.7 mm, vias 0 -> 1
- net Net-(D3-A): track 10.7 -> 0.00 mm, vias 1 -> 0
- net Net-(D1-K): track 0.00 -> 7.44 mm, vias 0 -> 1
- net Net-(D1-A): track 7.44 -> 0.00 mm, vias 1 -> 0
- net Net-(D2-K): track 0.00 -> 6.39 mm, vias 0 -> 1
- net Net-(D2-A): track 6.39 -> 0.00 mm, vias 1 -> 0
Changed lines of the file:
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@@
   (net 0 "")
   (net 1 "/BTN_ROW0")
-  (net 2 "Net-(D1-A)")
+  (net 2 "Net-(D1-K)")
   (net 3 "/BTN_ROW1")
-  (net 4 "Net-(D2-A)")
+  (net 4 "Net-(D2-K)")
   (net 5 "/BTN_ROW2")
-  (net 6 "Net-(D3-A)")
+  (net 6 "Net-(D3-K)")
   (net 7 "/BTN_COL")
   (net 8 "GND")
   (footprint "Diode_SMD:D_SOD-123" (layer "F.Cu")
-    (at 237.871 131.445)
+    (at 237.871 131.445 180)
     (descr "SOD-123")
     (tags "SOD-123")
@@
     (property "ki_keywords" "diode")
     (attr smd)
-    (fp_text reference "D3" (at 0 -1.778) (layer "F.SilkS")
+    (fp_text reference "D3" (at 0 1.905) (layer "F.SilkS")
         (effects (font (size 1 1) (thickness 0.15)))
     )
@@
     (fp_line (start 1.4 0.9) (end -1.4 0.9)
       (stroke (width 0.1) (type solid)) (layer "F.Fab"))
-    (pad "1" smd roundrect (at -1.65 0) (size 0.9 1.2) (layers "F.Cu" "F.Paste" "F.Mask") (roundrect_rratio 0.25)
-      (net 5 "/BTN_ROW2") (pinfunction "K") (pintype "passive"))
-    (pad "2" smd roundrect (at 1.65 0) (size 0.9 1.2) (layers "F.Cu" "F.Paste" "F.Mask") (roundrect_rratio 0.25)
-      (net 6 "Net-(D3-A)") (pinfunction "A") (pintype "passive"))
+    (pad "1" smd roundrect (at -1.65 0 180) (size 0.9 1.2) (layers "F.Cu" "F.Paste" "F.Mask") (roundrect_rratio 0.25)
+      (net 6 "Net-(D3-K)") (pinfunction "K") (pintype "passive"))
+    (pad "2" smd roundrect (at 1.65 0 180) (size 0.9 1.2) (layers "F.Cu" "F.Paste" "F.Mask") (roundrect_rratio 0.25)
+      (net 5 "/BTN_ROW2") (pinfunction "A") (pintype "passive"))
     (model "${KICAD6_3DMODEL_DIR}/Diode_SMD.3dshapes/D_SOD-123.wrl"
       (offset (xyz 0 0 0))
@@
       (net 7 "/BTN_COL") (pinfunction "1") (pintype "passive"))
     (pad "2" smd roundrect locked (at 4.060001 0 225) (size 1.7 2.7) (layers "F.Cu" "F.Paste" "F.Mask") (roundrect_rratio 0.25)
-      (net 6 "Net-(D3-A)") (pinfunction "2") (pintype "passive") (clearance 0.2794))
+      (net 6 "Net-(D3-K)") (pinfunction "2") (pintype "passive") (clearance 0.2794))
     (model ":ENYA_3DMOD:ENYA_Switch_Push.3dshapes/SKSTAJE010.step"
       (offset (xyz 0 0 0))
@@
   )
   (footprint "Diode_SMD:D_SOD-123" (layer "F.Cu")
-    (at 216.916 131.191 180)
+    (at 216.916 131.191)
     (descr "SOD-123")
     (tags "SOD-123")
@@
     (property "ki_keywords" "diode")
     (attr smd)
-    (fp_text reference "D1" (at -3.429 0) (layer "F.SilkS")
+    (fp_text reference "D1" (at 3.302 0) (layer "F.SilkS")
         (effects (font (size 1 1) (thickness 0.15)))
     )
@@
     (fp_line (start 1.4 0.9) (end -1.4 0.9)
       (stroke (width 0.1) (type solid)) (layer "F.Fab"))
-    (pad "1" smd roundrect (at -1.65 0 180) (size 0.9 1.2) (layers "F.Cu" "F.Paste" "F.Mask") (roundrect_rratio 0.25)
-      (net 1 "/BTN_ROW0") (pinfunction "K") (pintype "passive"))
-    (pad "2" smd roundrect (at 1.65 0 180) (size 0.9 1.2) (layers "F.Cu" "F.Paste" "F.Mask") (roundrect_rratio 0.25)
-      (net 2 "Net-(D1-A)") (pinfunction "A") (pintype "passive"))
+    (pad "1" smd roundrect (at -1.65 0) (size 0.9 1.2) (layers "F.Cu" "F.Paste" "F.Mask") (roundrect_rratio 0.25)
+      (net 2 "Net-(D1-K)") (pinfunction "K") (pintype "passive"))
+    (pad "2" smd roundrect (at 1.65 0) (size 0.9 1.2) (layers "F.Cu" "F.Paste" "F.Mask") (roundrect_rratio 0.25)
+      (net 1 "/BTN_ROW0") (pinfunction "A") (pintype "passive"))
     (model "${KICAD6_3DMODEL_DIR}/Diode_SMD.3dshapes/D_SOD-123.wrl"
       (offset (xyz 0 0 0))
@@
   )
   (footprint "Diode_SMD:D_SOD-123" (layer "F.Cu")
-    (at 222.504 121.92)
+    (at 222.504 121.92 180)
     (descr "SOD-123")
     (tags "SOD-123")
@@
     (property "ki_keywords" "diode")
     (attr smd)
-    (fp_text reference "D2" (at -3.429 0) (layer "F.SilkS")
+    (fp_text reference "D2" (at 3.302 0) (layer "F.SilkS")
         (effects (font (size 1 1) (thickness 0.15)))
     )
@@
     (fp_line (start 1.4 0.9) (end -1.4 0.9)
       (stroke (width 0.1) (type solid)) (layer "F.Fab"))
-    (pad "1" smd roundrect (at -1.65 0) (size 0.9 1.2) (layers "F.Cu" "F.Paste" "F.Mask") (roundrect_rratio 0.25)
-      (net 3 "/BTN_ROW1") (pinfunction "K") (pintype "passive"))
-    (pad "2" smd roundrect (at 1.65 0) (size 0.9 1.2) (layers "F.Cu" "F.Paste" "F.Mask") (roundrect_rratio 0.25)
-      (net 4 "Net-(D2-A)") (pinfunction "A") (pintype "passive"))
+    (pad "1" smd roundrect (at -1.65 0 180) (size 0.9 1.2) (layers "F.Cu" "F.Paste" "F.Mask") (roundrect_rratio 0.25)
+      (net 4 "Net-(D2-K)") (pinfunction "K") (pintype "passive"))
+    (pad "2" smd roundrect (at 1.65 0 180) (size 0.9 1.2) (layers "F.Cu" "F.Paste" "F.Mask") (roundrect_rratio 0.25)
+      (net 3 "/BTN_ROW1") (pinfunction "A") (pintype "passive"))
     (model "${KICAD6_3DMODEL_DIR}/Diode_SMD.3dshapes/D_SOD-123.wrl"
       (offset (xyz 0 0 0))
@@
       (net 7 "/BTN_COL") (pinfunction "1") (pintype "passive"))
     (pad "2" smd roundrect locked (at 4.06 0 270) (size 1.7 2.7) (layers "F.Cu" "F.Paste" "F.Mask") (roundrect_rratio 0.25)
-      (net 2 "Net-(D1-A)") (pinfunction "2") (pintype "passive"))
+      (net 2 "Net-(D1-K)") (pinfunction "2") (pintype "passive"))
     (model ":ENYA_3DMOD:ENYA_Switch_Push.3dshapes/SKSTAJE010.step"
       (offset (xyz 0 0 0))
@@
       (net 7 "/BTN_COL") (pinfunction "1") (pintype "passive"))
     (pad "2" smd roundrect locked (at 4.06 0 180) (size 1.7 2.7) (layers "F.Cu" "F.Paste" "F.Mask") (roundrect_rratio 0.25)
-      (net 4 "Net-(D2-A)") (pinfunction "2") (pintype "passive"))
+      (net 4 "Net-(D2-K)") (pinfunction "2") (pintype "passive"))
     (model ":ENYA_3DMOD:ENYA_Switch_Push.3dshapes/SKSTAJE010.step"
       (offset (xyz 0 0 0))
@@
       (net 7 "/BTN_COL") (pinfunction "1") (pintype "passive"))
     (pad "2" smd roundrect locked (at 4.06 0 180) (size 1.7 2.7) (layers "B.Cu" "B.Paste" "B.Mask") (roundrect_rratio 0.25)
-      (net 4 "Net-(D2-A)") (pinfunction "2") (pintype "passive"))
+      (net 4 "Net-(D2-K)") (pinfunction "2") (pintype "passive"))
     (model ":ENYA_3DMOD:ENYA_Switch_Push.3dshapes/SKSTAJE010.step"
       (offset (xyz 0 0 0))
@@
       (net 7 "/BTN_COL") (pinfunction "1") (pintype "passive"))
     (pad "2" smd roundrect locked (at 4.06 0 270) (size 1.7 2.7) (layers "B.Cu" "B.Paste" "B.Mask") (roundrect_rratio 0.25)
-      (net 2 "Net-(D1-A)") (pinfunction "2") (pintype "passive"))
+      (net 2 "Net-(D1-K)") (pinfunction "2") (pintype "passive"))
     (model ":ENYA_3DMOD:ENYA_Switch_Push.3dshapes/SKSTAJE010.step"
       (offset (xyz 0 0 0))
@@
       (net 7 "/BTN_COL") (pinfunction "1") (pintype "passive"))
     (pad "2" smd roundrect locked (at 4.060001 0 225) (size 1.7 2.7) (layers "B.Cu" "B.Paste" "B.Mask") (roundrect_rratio 0.25)
-      (net 6 "Net-(D3-A)") (pinfunction "2") (pintype "passive") (clearance 0.2794))
+      (net 6 "Net-(D3-K)") (pinfunction "2") (pintype "passive") (clearance 0.2794))
     (model ":ENYA_3DMOD:ENYA_Switch_Push.3dshapes/SKSTAJE010.step"
       (offset (xyz 0 0 0))

Commit message: WIP
Connections:
- J1 pad 1: /BTN_COL -> GND
- J1 pad 2: /BTN_ROW0 -> /BTN_ROW2
- J1 pad 4: /BTN_ROW2 -> /BTN_ROW0
- J1 pad 5: GND -> /BTN_COL
- J2 pad 1: /BTN_COL -> GND
- J2 pad 2: /BTN_ROW0 -> /BTN_ROW2
- J2 pad 4: /BTN_ROW2 -> /BTN_ROW0
- J2 pad 5: GND -> /BTN_COL
Routing:
- net /BTN_ROW2: track 41.0 -> 41.4 mm, vias 3 -> 4
- net GND: vias 61 -> 63
